File: NixiePowerSupply.sch (KiCad schematic (older format))
At the start: 17 parts, among them J1 BARREL_JACK, P1 CONN_01X03, P2 CONN_01X02, T1 IRF644, U1 MAX1771

Commit message: Trying to make a new board
Parts:
- P2: footprint (none) -> nixie:Pin_Header_Straight_1x03_Pitch2.54mm_No_Center
Changed lines of the file:
@@
 F 0 "P2" H 9050 3850 50  0000 C CNN
 F 1 "CONN_01X02" V 9150 3700 50  0000 C CNN
-F 2 "" H 9050 3700 50  0000 C CNN
+F 2 "nixie:Pin_Header_Straight_1x03_Pitch2.54mm_No_Center" H 9050 3700 50  0001 C CNN
 F 3 "" H 9050 3700 50  0000 C CNN
 	1    9050 3700
